File: boilerplate/esp32/esp32_boilerplate.kicad_pcb (KiCad board)
At the start: 2 copper layers, 100 x 100 mm, 15 parts, among them SW1 TS-1187A-B-A-B, SW2 TS-1187A-B-A-B, U1 CH340C_C7464026, U2 AMS1117-3.3, U3 ESP32-WROOM-32E(8MB)

Commit message: Routed ESP32 boilerplate
Signed-off-by: Pablo Garrido <pablogs9@gmail.com>
Parts:
- added LED3: WS2812B-B, easyeda2kicad:LED-SMD_4P-L5.0-W5.0-BL_TC5050RGB, F.Cu at (141.8, 62.5)
- moved R3 4.41 mm to (111.5, 71.5), turned to 180 degrees
- moved R1 4.27 mm to (118.9, 56.8)
- moved R2 4.27 mm to (124.5, 56.8)
- moved U1 4.27 mm to (121.8, 63.1)
- moved USBC1 4.27 mm to (122.0, 52.4)
- moved C1 4.27 mm to (116.7, 66.7)
- moved LED2 3.68 mm to (107.8, 69.2)
- moved C2 3.18 mm to (132.4, 54.4)
- moved C3 3.18 mm to (132.4, 66.4)
- moved U2 3.18 mm to (132.4, 60.5)
- moved R7 2.44 mm to (111.5, 69.2), turned to 180 degrees
Routing:
- net /3V3: track 11.7 -> 67.4 mm
- net /ESP_RXD: track 0.00 -> 43.3 mm, vias 0 -> 2
- net /ESP_TXD: track 0.00 -> 42.8 mm, vias 0 -> 2
- net /ESP_EN: track 0.00 -> 33.5 mm, vias 0 -> 2
- net /ESP_LED: track 0.00 -> 17.1 mm, vias 0 -> 2
- net /5V: track 3.51 -> 18.9 mm
- net /ESP_PROG: track 0.00 -> 12.3 mm
- net /USB_P: track 0.00 -> 11.4 mm
- net /USB_N: track 0.00 -> 9.09 mm
- net Net-(LED2-K): track 0.00 -> 2.15 mm
- net Net-(LED1-K): track 0.00 -> 2.14 mm
- net GND: track 0.00 -> 2.07 mm
Other:
- board size 100 x 100 mm -> 66.7 x 27.3 mm
