File: boilerplate/esp32/esp32_boilerplate.kicad_sch (KiCad schematic)
At the start: 15 parts, among them SW1 TS-1187A-B-A-B, SW2 TS-1187A-B-A-B, U1 CH340C_C7464026, U2 AMS1117-3.3, U3 ESP32-WROOM-32E(8MB)

Commit message: Routed ESP32 boilerplate
Signed-off-by: Pablo Garrido <pablogs9@gmail.com>
Parts:
- added LED3: WS2812B-B, easyeda2kicad:LED-SMD_4P-L5.0-W5.0-BL_TC5050RGB, symbol easyeda2kicad:WS2812B-B
Changed lines of the file:
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@@
+	)
+	(symbol
+		(lib_id "easyeda2kicad:WS2812B-B")
+		(at 214.63 119.38 0)
+		(unit 1)
+		(exclude_from_sim no)
+		(in_bom yes)
+		(on_board yes)
+		(dnp no)
+		(fields_autoplaced yes)
+		(property "Reference" "LED3"
+			(at 214.63 110.49 0)
+			(effects
+				(font
+					(size 1.27 1.27)
+				)
+			)
+		)
+		(property "Value" "WS2812B-B"
+			(at 214.63 113.03 0)
+			(effects
+				(font
+					(size 1.27 1.27)
+				)
+			)
+		)
+		(property "Footprint" "easyeda2kicad:LED-SMD_4P-L5.0-W5.0-BL_TC5050RGB"
+			(at 214.63 128.27 0)
+			(effects
+				(font
+					(size 1.27 1.27)
+				)
+				(hide yes)
+			)
+		)
+		(property "Datasheet" "https://lcsc.com/product-detail/Light-Emitting-Diodes-LED_5050-RGBIntegrated-Light-4Pin_C114586.html"
+			(at 214.63 130.81 0)
+			(effects
+				(font
+					(size 1.27 1.27)
+				)
+				(hide yes)
+			)
+		)
+		(property "Description" ""
+			(at 214.63 119.38 0)
+			(effects
+				(font
+					(size 1.27 1.27)
+				)
+				(hide yes)
+			)
+		)
+		(property "LCSC Part" "C114586"
+			(at 214.63 133.35 0)
+			(effects
+				(font
+					(size 1.27 1.27)
+				)
+				(hide yes)
+			)
+		)
+		(pin "1"
+		)
+		(pin "2"
+		)
+		(pin "4"
+		)
+		(pin "3"
+		)
+		(instances
+			(project ""
+				(path "/94e27b1b-416d-4c0f-a1ba-3839408eff47"
+					(reference "LED3")
+					(unit 1)
+				)
+			)
+		)
 	)
 	(symbol
