File: kicad_makespace_tutorial.kicad_pcb (KiCad board)
At the start: 2 copper layers, 64.5 x 22.5 mm, 42 parts, among them J1 Screw_Terminal_01x02, J2 Conn_01x08_Pin, SW1 TS-1187A-B-A-B, SW2 TS-1187A-B-A-B, U1 AMS1117-3.3, U2 CH340C_C7464026, U3 ESP32-WROOM-32E(8MB), U4 MAX98357AETE+T

Commit message: Bump Desing
Parts:
- removed C4: 10u, easyeda2kicad:C1206
- removed C5: 0.1u, easyeda2kicad:C0603
- removed R1, R2: 5k1, easyeda2kicad:R0603
- removed R7: 100, easyeda2kicad:R0603
- removed SW1, SW2: TS-1187A-B-A-B, easyeda2kicad:SW-SMD_4P-L5.1-W5.1-P3.70-LS6.5-TL_H1.5
- removed TP10, TP11, TP7, TP8, TP9: TestPoint, TestPoint:TestPoint_Pad_D1.0mm
- added C6: 0.1u, easyeda2kicad:C0805, F.Cu at (118.5, 119.5)
- added J3: Conn_02x03_Counter_Clockwise, Connector_PinHeader_2.00mm:PinHeader_2x03_P2.00mm_Vertical, F.Cu at (130.0, 104.5)
- added JP4: SolderJumper_2_Open, Jumper:SolderJumper-2_P1.3mm_Open_TrianglePad1.0x1.5mm, B.Cu at (113.9, 112.0)
- added JP5: SolderJumper_2_Open, Jumper:SolderJumper-2_P1.3mm_Open_TrianglePad1.0x1.5mm, B.Cu at (111.3, 112.0)
- added LED3: WS2812B-2020, easyeda2kicad:LED-SMD_4P-L2.0-W2.0-TL_WS2812B-2020, F.Cu at (103.5, 114.9)
- added LED4: WS2812B-2020, easyeda2kicad:LED-SMD_4P-L2.0-W2.0-TL_WS2812B-2020, F.Cu at (116.4, 119.8)
- added LED5: WS2812B-2020, easyeda2kicad:LED-SMD_4P-L2.0-W2.0-TL_WS2812B-2020, F.Cu at (135.2, 108.0)
- added R8: 100, easyeda2kicad:R0805, F.Cu at (113.5, 110.7)
- added TP15: TestPoint, TestPoint:TestPoint_Pad_D1.0mm, B.Cu at (86.5, 107.0)
- added TP16: TestPoint, TestPoint:TestPoint_Pad_D1.0mm, B.Cu at (84.5, 107.0)
- added TP17: TestPoint, TestPoint:TestPoint_Pad_D1.0mm, B.Cu at (85.5, 108.8)
- added TP18: TestPoint, TestPoint:TestPoint_Pad_D1.0mm, B.Cu at (99.0, 102.0)
- added TP19: TestPoint, TestPoint:TestPoint_Pad_D1.0mm, B.Cu at (97.0, 102.0)
- added U5: ESP32-S3-WROOM-1-N4R2, easyeda2kicad:WIRELM-SMD_ESP32-S3-WROOM-1, F.Cu at (91.9, 111.0)
- C3: value 0.1u -> 10u; footprint easyeda2kicad:C0603 -> easyeda2kicad:C0805
- LED1: value KT-0603R -> FC-2012HRK-620D; footprint easyeda2kicad:LED0603-RD -> easyeda2kicad:LED0805-R-RD
- LED2: value KT-0603R -> XL-2012UGC; footprint easyeda2kicad:LED0603-RD -> easyeda2kicad:LED0805-RD_GREEN
- R3: footprint easyeda2kicad:R0603 -> easyeda2kicad:R0805
- U2: value CH340C_C7464026 -> 5k1; footprint easyeda2kicad:SOP-16_L10.0-W3.9-P1.27-LS6.0-BL -> easyeda2kicad:R0805
- U3: value ESP32-WROOM-32E(8MB) -> 5k1; footprint easyeda2kicad:WIFI-SMD_ESP32-WROOM-32E -> easyeda2kicad:R0805
- moved U3 18.3 mm to (109.9, 108.7), turned to 180 degrees
- moved R3 9.63 mm to (113.5, 112.4), turned to 180 degrees
- moved C3 9.56 mm to (125.6, 115.9), turned to 0 degrees
- moved G*** 9.50 mm to (111.9, 119.6)
- moved U2 9.42 mm to (105.0, 108.7), turned to 0 degrees
- moved LED1 5.70 mm to (109.7, 110.8), turned to 180 degrees
- moved LED2 3.99 mm to (109.7, 112.5), turned to 180 degrees
Connections:
- C3 pad 1: GND -> /5V
- C3 pad 2: /3V3 -> GND
- LED1 pad 1: Net-(LED1-K) -> /ESP_LED
- LED1 pad 2: /ESP_LED -> Net-(LED1--)
- R3 pad 2: Net-(LED1-K) -> Net-(LED2-K)
- U2 pad 2: /ESP_RXD -> Net-(USBC1-CC2)
- U3 pad 2: /3V3 -> Net-(USBC1-CC1)
- USBC1 pad 1: GND -> (no net)
- USBC1 pad 2: GND -> (no net)
- USBC1 pad 3: GND -> (no net)
Routing:
- net /ESP_EN: track 56.1 -> 0.00 mm, vias 2 -> 0
- net /WLED_VDD: track 0.00 -> 53.6 mm, vias 0 -> 3
- net /GPIO_19: track 3.10 -> 46.5 mm
- net /GPIO_16: track 8.22 -> 50.7 mm
- net Net-(LED4-DO): track 0.00 -> 41.5 mm, vias 0 -> 2
- net /ESP_PROG: track 41.9 -> 3.55 mm, vias 2 -> 1
- net /GPIO_4: track 8.21 -> 46.0 mm
- net /GPIO_17: track 8.62 -> 43.0 mm
- net /ESP_TXD: track 30.5 -> 5.73 mm, vias 2 -> 1
- net /ESP_RXD: track 29.5 -> 5.42 mm, vias 2 -> 1
- net Net-(LED3-DO): track 0.00 -> 14.9 mm, vias 0 -> 2
- net /3V3: track 87.5 -> 79.8 mm, vias 6 -> 5
- net /SD_MODE: track 38.0 -> 31.6 mm, vias 1 -> 3
- net /I2S_LRCLK: track 30.2 -> 24.6 mm, vias 2 -> 0
- net /USB_P: track 15.2 -> 19.9 mm
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
Commit message: Final design
Signed-off-by: Pablo Garrido <pablogs9@gmail.com>
Parts:
- added R1: 100, easyeda2kicad:R0805, F.Cu at (111.1, 114.2)
- moved LED3 0.10 mm to (103.4, 114.9)
Routing:
- net /ESP_EN: track 0.00 -> 34.1 mm, vias 0 -> 2
- net /3V3: track 79.8 -> 82.1 mm
- net /GPIO_19: track 46.5 -> 47.0 mm
- net /USB_P: track 19.9 -> 20.4 mm

Commit message: Final Updates
Parts:
- removed JP4, JP5: SolderJumper_2_Open, Jumper:SolderJumper-2_P1.3mm_Open_TrianglePad1.0x1.5mm
- added JP6: Jumper_3_Bridged12, Jumper:SolderJumper-3_P1.3mm_Bridged2Bar12_RoundedPad1.0x1.5mm_NumberLabels, B.Cu at (112.5, 111.1)
- J3: footprint Connector_PinHeader_2.00mm:PinHeader_2x03_P2.00mm_Vertical -> Connector_PinHeader_2.54mm:PinHeader_2x03_P2.54mm_Vertical
- R4: moved to F.Cu
- moved R4 5.80 mm to (131.2, 110.2), turned to 0 degrees
- moved J3 0.50 mm to (130.0, 105.0)
Connections:
- J2 pad 7: /GPIO_35 -> /GPIO_16
- J3 pad 5: /GPIO_4 -> /GPIO_34
- U5 pad 29: /GPIO_4 -> unconnected-(U5-IO36-Pad29)
- U5 pad 30: /GPIO_16 -> unconnected-(U5-IO37-Pad30)
- U5 pad 7: /GPIO_35 -> /GPIO_16
Routing:
- net /GPIO_34: track 2.77 -> 67.6 mm
- net /GPIO_4: track 46.1 -> 0.00 mm, vias 1 -> 0
- net /GPIO_16: track 50.9 -> 76.2 mm, vias 1 -> 3
- net /5V: track 78.9 -> 84.7 mm, vias 5 -> 6
- net /GPIO_35: track 4.74 -> 0.00 mm, vias 1 -> 0
- net /3V3: track 82.1 -> 80.3 mm
- net /GPIO_19: track 47.0 -> 48.2 mm
- net /ESP_EN: track 34.1 -> 35.0 mm
- net /SD_MODE: track 31.5 -> 31.3 mm, vias 3 -> 4
- net GND: vias 43 -> 45
