File: kicad_makespace_tutorial.kicad_sch (KiCad schematic)
At the start: 41 parts, among them J1 Screw_Terminal_01x02, J2 Conn_01x08_Pin, SW1 TS-1187A-B-A-B, SW2 TS-1187A-B-A-B, U1 AMS1117-3.3, U2 CH340C_C7464026, U3 ESP32-WROOM-32E(8MB), U4 MAX98357AETE+T

Commit message: Bump Desing
Parts:
- removed C3, C5: 0.1u, easyeda2kicad:C0603, symbol easyeda2kicad:CC0603KRX7R9BB104
- removed C4: 10u, easyeda2kicad:C1206, symbol easyeda2kicad:CL31A106KBHNNNE
- removed LED1, LED2: KT-0603R, easyeda2kicad:LED0603-RD, symbol easyeda2kicad:KT-0603R
- removed R1, R2: 5k1, easyeda2kicad:R0603, symbol easyeda2kicad:0603WAF5101T5E
- removed R3, R7: 100, easyeda2kicad:R0603, symbol easyeda2kicad:0603WAF1000T5E
- removed SW1, SW2: TS-1187A-B-A-B, easyeda2kicad:SW-SMD_4P-L5.1-W5.1-P3.70-LS6.5-TL_H1.5, symbol easyeda2kicad:TS-1187A-B-A-B
- removed TP10, TP11, TP7, TP8, TP9: TestPoint, TestPoint:TestPoint_Pad_D1.0mm, symbol Connector:TestPoint
- removed U2: CH340C_C7464026, easyeda2kicad:SOP-16_L10.0-W3.9-P1.27-LS6.0-BL, symbol easyeda2kicad:CH340C_C7464026
- removed U3: ESP32-WROOM-32E(8MB), easyeda2kicad:WIFI-SMD_ESP32-WROOM-32E, symbol easyeda2kicad:ESP32-WROOM-32E(8MB)
- added C3: 10u, easyeda2kicad:C0805, symbol easyeda2kicad:CL21A106KAYNNNE
- added C6: 0.1u, easyeda2kicad:C0805, symbol easyeda2kicad:CC0805KRX7R9BB104
- added J3: Conn_02x03_Counter_Clockwise, Connector_PinHeader_2.00mm:PinHeader_2x03_P2.00mm_Vertical, symbol Connector_Generic:Conn_02x03_Counter_Clockwise
- added JP4, JP5: SolderJumper_2_Open, Jumper:SolderJumper-2_P1.3mm_Open_TrianglePad1.0x1.5mm, symbol Jumper:SolderJumper_2_Open
- added LED1: FC-2012HRK-620D, easyeda2kicad:LED0805-R-RD, symbol easyeda2kicad:FC-2012HRK-620D
- added LED2: XL-2012UGC, easyeda2kicad:LED0805-RD_GREEN, symbol easyeda2kicad:XL-2012UGC
- added LED3, LED4, LED5: WS2812B-2020, easyeda2kicad:LED-SMD_4P-L2.0-W2.0-TL_WS2812B-2020, symbol easyeda2kicad:WS2812B-2020
- added R3, R8: 100, easyeda2kicad:R0805, symbol easyeda2kicad:0805W8F1000T5E
- added TP15, TP16, TP17, TP18, TP19: TestPoint, TestPoint:TestPoint_Pad_D1.0mm, symbol Connector:TestPoint
- added U2, U3: 5k1, easyeda2kicad:R0805, symbol easyeda2kicad:FRC0805J512TS
- added U5: ESP32-S3-WROOM-1-N4R2, easyeda2kicad:WIRELM-SMD_ESP32-S3-WROOM-1, symbol easyeda2kicad:ESP32-S3-WROOM-1-N4R2
Connections:
- net 3V3: now also JP5.2 (B), LED2.2 (A), U5.2 (3V3)
- net 5V: now also C3.1, C6.2, JP4.2 (B)
- net ESP_EN: now also U5.3 (EN)
- net ESP_LED: now also LED1.1 (+), U5.24 (IO47)
- net ESP_PROG: now also TP18.1, U5.27 (IO0)
- net ESP_RXD: now also TP15.1, U5.36 (RXD0)
- net ESP_TXD: now also TP16.1, U5.37 (TXD0)
- net GND: now also C3.2, C6.1, J3.3 (Pin_3), J3.4 (Pin_4), LED3.2 (GND), LED4.2 (GND), LED5.2 (GND), R3.1, R8.1, TP17.1, TP19.1, U2.1, U3.1, U5.1 (GND), U5.40 (GND), U5.41 (EPAD)
- net GPIO_16: now also J3.6 (Pin_6), U5.30 (IO37)
- net GPIO_17: now also J3.2 (Pin_2), U5.31 (IO38)
- net GPIO_18: now also U5.33 (IO40)
- net GPIO_19: now also J3.1 (Pin_1), U5.34 (IO41)
- net GPIO_21: now also U5.35 (IO42)
- net GPIO_25: now also U5.10 (IO17)
- net GPIO_26: now also U5.11 (IO18)
- net GPIO_32: now also U5.8 (IO15)
- net GPIO_33: now also U5.9 (IO16)
- net GPIO_34: now also U5.6 (IO6)
- net GPIO_35: now also U5.7 (IO7)
- net GPIO_4: now also J3.5 (Pin_5), U5.29 (IO36)
- net GPIO_5: now also U5.32 (IO39)
- net I2S_BCLK: now also U5.20 (IO12)
- net I2S_DIN: now also U5.19 (IO11)
- net I2S_LRCLK: now also U5.21 (IO13)
- net USB_N: now also U5.13 (IO19)
- net USB_P: now also U5.14 (IO20)
- net at USBC1.B5 (CC2): now also U2.2
- net at USBC1.A5 (CC1): now also U3.2
- new net: LED3.1 (DO), LED4.3 (DI)
- new net: LED2.1 (K), R3.2
- new net: LED1.2 (-), R8.2
- new net: LED4.1 (DO), LED5.3 (DI)
- new net WLED: LED3.3 (DI), U5.18 (IO10)
- new net WLED_VDD: JP4.1 (A), JP5.1 (A), LED3.4 (VDD), LED4.4 (VDD), LED5.4 (VDD)
Other:
- note added: "WLED"
- note removed: "USB-UART Bridge"
- moved on the sheet: C1, C2, H1, H3, J1, J2, R4, R5, R6, U1, U4, USBC1

Commit message: Final design
Signed-off-by: Pablo Garrido <pablogs9@gmail.com>
Parts:
- added R1: 100, easyeda2kicad:R0805, symbol easyeda2kicad:0805W8F1000T5E
Connections:
- net 3V3: now also R1.2
- net ESP_EN: now also R1.1
Changed lines of the file:
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@@
 	)
 	(junction
+		(at 165.1 151.13)
+		(diameter 0)
+		(color 0 0 0 0)
+	)
+	(junction
 		(at 337.82 81.28)
 		(diameter 0)
@@
 	(wire
 		(pts
-			(xy 179.07 151.13) (xy 193.04 151.13)
+			(xy 156.21 151.13) (xy 165.1 151.13)
 		)
 		(stroke
@@
 	(wire
 		(pts
+			(xy 165.1 138.43) (xy 165.1 140.97)
+		)
+		(stroke
+			(width 0)
+			(type default)
+		)
+	)
+	(wire
+		(pts
 			(xy 219.71 124.46) (xy 215.9 124.46)
 		)
@@
 	(wire
 		(pts
+			(xy 165.1 151.13) (xy 193.04 151.13)
+		)
+		(stroke
+			(width 0)
+			(type default)
+		)
+	)
+	(wire
+		(pts
 			(xy 219.71 116.84) (xy 215.9 116.84)
 		)
@@
 	)
 	(label "ESP_EN"
-		(at 179.07 151.13 0)
+		(at 156.21 151.13 0)
 		(effects
 			(font
@@
 		)
 	)
+	(label "3V3"
+		(at 165.1 138.43 0)
+		(effects
+			(font
+				(size 1.27 1.27)
+			)
+			(justify left bottom)
+		)
+	)
 	(label "ESP_LED"
 		(at 219.71 111.76 0)
@@
 					(unit 1)
 				)
+			)
+		)
+	)
+	(symbol
+		(lib_id "easyeda2kicad:0805W8F1000T5E")
+		(at 165.1 146.05 90)
+		(unit 1)
+		(exclude_from_sim no)
+		(in_bom yes)
+		(on_board yes)
+		(dnp no)
+		(fields_autoplaced yes)
+		(property "Reference" "R1"
+			(at 167.64 144.7799 90)
+			(effects
+				(font
+					(size 1.27 1.27)
+				)
+				(justify right)
+			)
+		)
+		(property "Value" "100"
+			(at 167.64 147.3199 90)
+			(effects
+				(font
+					(size 1.27 1.27)
+				)
+				(justify right)
+			)
+		)
+		(property "Footprint" "easyeda2kicad:R0805"
+			(at 172.72 146.05 0)
+			(effects
+				(font
+					(size 1.27 1.27)
+				)
+				(hide yes)
+			)
+		)
+		(property "Datasheet" "https://lcsc.com/product-detail/Chip-Resistor-Surface-Mount-UniOhm_100R-1000-1_C17408.html"
+			(at 175.26 146.05 0)
+			(effects
+				(font
+					(size 1.27 1.27)
+				)
+				(hide yes)
+			)
+		)
+		(property "Description" ""
+			(at 165.1 146.05 0)
+			(effects
+				(font
+					(size 1.27 1.27)
+				)
+				(hide yes)
+			)
+		)
+		(property "LCSC Part" "C17408"
+			(at 177.8 146.05 0)
+			(effects
+				(font
+					(size 1.27 1.27)
+				)
+				(hide yes)
+			)
+		)
+		(pin "2"
+		)
+		(pin "1"
+		)
+		(instances
+			(project "kicad_makespace_tutorial"
+				(path "/6e6169dc-bc5d-4a4e-95fd-65529ef4ae3e"
+					(reference "R1")
+					(unit 1)
+				)

Commit message: Final Updates
Parts:
- J3: footprint Connector_PinHeader_2.00mm:PinHeader_2x03_P2.00mm_Vertical -> Connector_PinHeader_2.54mm:PinHeader_2x03_P2.54mm_Vertical
Connections:
- net GPIO_35 is gone; now on net GPIO_16: J2.7 (Pin_7), U5.7 (IO7)
- net GPIO_16: no longer U5.30 (IO37)
- net GPIO_34: now also J3.5 (Pin_5)
- net GPIO_4: no longer names the net of U5.29 (IO36)
- net GPIO_4: no longer J3.5 (Pin_5)
Other:
- note added: "RENAME NETS WITH WRONG GPIO AND DO NOT USE PROTECTED GPIOS!!!"
Changed lines of the file:
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@@
 (kicad_sch
-	(version 20231120)
+	(version 20250114)
 	(generator "eeschema")
-	(generator_version "8.0")
+	(generator_version "9.0")
 	(paper "A3")
 	(title_block
@@
 		(company "Casa Cactus")
 	)
+	(text "Button & LEDs"
+		(exclude_from_sim no)
+		(at 345.186 189.738 0)
+		(effects
+			(font
+				(size 1.778 1.778)
+				(thickness 0.3556)
+				(bold yes)
+			)
+		)
+	)
+	(text "Mounting Holes"
+		(exclude_from_sim no)
+		(at 48.006 247.396 0)
+		(effects
+			(font
+				(size 1.778 1.778)
+				(thickness 0.3556)
+				(bold yes)
+			)
+		)
+	)
+	(text "Power Stage"
+		(exclude_from_sim no)
+		(at 208.026 25.908 0)
+		(effects
+			(font
+				(size 1.778 1.778)
+				(thickness 0.3556)
+				(bold yes)
+			)
+		)
+	)
+	(text "GPIO"
+		(exclude_from_sim no)
+		(at 215.392 240.03 0)
+		(effects
+			(font
+				(size 1.778 1.778)
+				(thickness 0.3556)
+				(bold yes)
+			)
+		)
+	)
+	(text "Audio Subsystem"
+		(exclude_from_sim no)
+		(at 341.376 24.638 0)
+		(effects
+			(font
+				(size 1.778 1.778)
+				(thickness 0.3556)
+				(bold yes)
+			)
+		)
+	)
+	(text "RENAME NETS WITH WRONG GPIO AND DO NOT USE PROTECTED GPIOS!!!"
+		(exclude_from_sim no)
+		(at 211.074 132.334 0)
+		(effects
+			(font
+				(size 5.08 5.08)
+				(color 255 0 0 1)
+			)
+		)
+	)
+	(text "ESP32"
+		(exclude_from_sim no)
+		(at 203.962 98.806 0)
+		(effects
+			(font
+				(size 1.778 1.778)
+				(thickness 0.3556)
+				(bold yes)
+			)
+		)
+	)
+	(text "WLED"
+		(exclude_from_sim no)
+		(at 344.678 125.222 0)
+		(effects
+			(font
+				(size 1.778 1.778)
+				(thickness 0.3556)
+				(bold yes)
+			)
+		)
+	)
+	(text "USB Connector"
+		(exclude_from_sim no)
+		(at 69.088 20.32 0)
+		(effects
+			(font
+				(size 1.778 1.778)
+				(thickness 0.3556)
+				(bold yes)
+			)
+		)
+	)
 	(junction
 		(at 318.77 62.23)
@@
 	(wire
 		(pts
-			(xy 179.07 140.97) (xy 193.04 140.97)
+			(xy 176.53 140.97) (xy 193.04 140.97)
 		)
 		(stroke
@@
 	(wire
 		(pts
-			(xy 179.07 143.51) (xy 193.04 143.51)
+			(xy 176.53 143.51) (xy 193.04 143.51)
 		)
 		(stroke
@@
 			"gASQgB0QQIVuB42IVUACSAAJIAEkgAodZQAJIAEkgASQgB0QQIVuB42IVUACSAAJIAEkgAodZQAJ"
 			"IAEkgASQgB0QQIVuB42IVUACSAAJIAEkgAodZQAJIAEkgASQgB0QQIVuB42IVUACSAAJIAEk8H/w"
-			"e4+QFN7h7AAAAABJRU5ErkJggg=="
-		)
-	)
-	(text "Button & LEDs"
-		(exclude_from_sim no)
-		(at 345.186 189.738 0)
-		(effects
-			(font
-				(size 1.778 1.778)
-				(thickness 0.3556)
-				(bold yes)
-			)
-		)
-	)
-	(text "Mounting Holes"
-		(exclude_from_sim no)
-		(at 48.006 247.396 0)
-		(effects
-			(font
-				(size 1.778 1.778)
-				(thickness 0.3556)
-				(bold yes)
-			)
-		)
-	)
-	(text "Power Stage"
-		(exclude_from_sim no)
-		(at 208.026 25.908 0)
-		(effects
-			(font
-				(size 1.778 1.778)
-				(thickness 0.3556)
-				(bold yes)
-			)
-		)
-	)
-	(text "GPIO"
-		(exclude_from_sim no)
-		(at 215.392 240.03 0)
-		(effects
-			(font
-				(size 1.778 1.778)
-				(thickness 0.3556)
-				(bold yes)
-			)
-		)
-	)
-	(text "Audio Subsystem"
-		(exclude_from_sim no)
-		(at 341.376 24.638 0)
-		(effects
-			(font
-				(size 1.778 1.778)
-				(thickness 0.3556)
-				(bold yes)
-			)
-		)
-	)
-	(text "ESP32"
-		(exclude_from_sim no)
-		(at 203.962 98.806 0)
-		(effects
-			(font
-				(size 1.778 1.778)
-				(thickness 0.3556)
-				(bold yes)
-			)
-		)
-	)
-	(text "WLED"
-		(exclude_from_sim no)
-		(at 344.678 125.222 0)
-		(effects
-			(font
-				(size 1.778 1.778)
-				(thickness 0.3556)
-				(bold yes)
-			)
-		)
-	)
-	(text "USB Connector"
-		(exclude_from_sim no)
-		(at 69.088 20.32 0)
-		(effects
-			(font
-				(size 1.778 1.778)
-				(thickness 0.3556)
-				(bold yes)
-			)
+			"e4+QFN7h7AAAAABJRU5ErkJgggAAAAAAAAAAAAAAAAAAAAAAAAAAAAAAAAAAAAAAAAAAAAAAAAAA"
+			"AAAAAAAAAAAAAAAAAAAAAAAAAAAAAAAAAAAAAAAAAAAAAAAAAAAAAAAAAAAAAAAAAAAAAAAAAAAA"
+			"AAAAAAAAAAAAAAAAAAAAAAAAAAAAAAAAAAAAAAAAAAAAAAAAAAAAAAAAAAAAAAAAAAAAAAAAAAAA"
+			"AAAAAAAAAAAAAAAAAAAAAAAAAAAAAAAAAAAAAAAAAAAAAAAAAAAAAAAAAAAAAAAAAAAAAAAAAAAA"
+			"AAAAAAAAAAAAAAAAAAAAAAAAAAAAAAAAAAAAAAAAAAAAAAAAAAAAAAAAAAAAAAAAAAAAAAAAAAAA"
+			"AAAAAAAAAAAAAAAAAAAAAAAAAAAAAAAAAAAAAAAAAAAAAAAAAAAAAAAAAAAAAAAAAAAAAAAAAAAA"
+			"AAAAAAAAAAAAAAAAAAAAAAAAAAAAAAAAAAAAAAAAAAAAAAAAAAAAAAAAAAAAAAAAAAAAAAAAAAAA"
+			"AAAAAAAAAAAAAAAAAAAAAAAAAAAAAAAAAAAAAAAAAAAAAAAAAAAAAAAAAAAAAAAAAAAAAAAAAAAA"
+			"AAAAAAAAAAAAAAAAAAAAAAAAAAAAAAAAAAAAAAAAAAAAAAAAAAAAAAAAAAAAAAAAAAAAAAAAAAAA"
+			"AAAAAAAAAAAAAAAAAAAAAAAAAAAAAAAAAAAAAAAAAAAAAAAAAAAAAAAAAAAAAAAAAAAAAAAAAAAA"
+			"AAAAAAAAAAAAAAAAAAAAAAAAAAAAAAAAAAAAAAAAAAAAAAAAAAAAAAAAAAAAAAAAAAAAAAAAAAAA"
+			"AAAAAAAAAAAAAAAAAAAAAAAAAAAAAAAAAAAAAAAAAAAAAAAAAAAAAAAAAAAAAAAAAAAAAAAAAAAA"
+			"AAAAAAAAAAAAAAAAAAAAAAAAAAAAAAAAAAAAAAAAAAAAAAAAAAAAAAAAAAAAAAAAAAAAAAAAAAAA"
+			"AAAAAAAAAAAAAAAAAAAAAAAAAAAAAAAAAAAAAAAAAAAAAAAAAAAAAAAAAAAAAAAAAAAAAAAAAAAA"
+			"AAAAAAAAAAAAAAAAAAAAAAAAAAAAAAAAAAAAAAAAAAAAAAAAAAAAAAAAAAAAAAAAAAAAAAAAAAAA"
+			"AAAAAAAAAAAAAAAAAAAAAAAAAAAAAAAAAAAAAAAAAAAAAAAAAAAAAAAAAAAAAAAAAAAAAAAAAAAA"
+			"AAAAAAAAAAAAAAAAAAAAAAAAAAAAAAAAAAAAAAAAAAAAAAAAAAAAAAAAAAAAAAAAAAAAAAAAAAAA"
+			"AAAAAAAAAAAAAAAAAAAAAAAAAAAAAAAAAAAAAAAAAAAAAAAAAAAAAAAAAAAAAAAAAAAAAAAAAAAA"
+			"AAAAAAAAAAAAAAAAAAAAAAAAAEABbW9KVgAAQDWxcEpWAACAV+ZuSlYAAADmWXBKVgAAAAAAAAAA"
+			"AACAiENwSlYAAAAAAAAAAAAAQGwrcEpWAAAAAAAAAAAAAMBJ429KVgAAwEIeeUpWAACAAW1vSlYA"
+			"AMAO8XlKVgAAgJPmbkpWAAAAAAAAAAAAAAAAAAAAAAAAwIhDcEpWAAAAAAAAAAAAAIBsK3BKVgAA"
+			"AAAAAAAAAABASuNvSlYAAABDHnlKVgAAwAFtb0pWAACAD/F5SlYAAMCU5m5KVgAAwOZZcEpWAAAA"
+			"AAAAAAAAAACJQ3BKVgAAAAAAAAAAAADAbCtwSlYAAAAAAAAAAAAAQEMeeUpWAAAAAAAAAAAAAAAC"
+			"bW9KVgAAQA/xeUpWAACAVuZuSlYAAADnWXBKVgAAAAAAAAAAAAAAAAAAAAAAAAAAAAAAAAAAAG0r"
+			"cEpWAAAAAAAAAAAAAEBL429KVgAAAEEeeUpWAABAAm1vSlYAAICXsXBKVgAAwJHmbkpWAABA51lw"
+			"SlYAAAAAAAAAAAAAwIlDcEpWAAAAAAAAAAAAAIBdKXBKVgAAAAAAAAAAAACAS+NvSlYAAMBBHnlK"
+			"VgAAgAJtb0pWAACArPB5SlYAAIBV5m5KVgAAgOdZcEpWAAAAAAAAAAAAAACKQ3BKVgAAAAAAAAAA"
+			"AABAXSlwSlYAAAAAAAAAAAAAAO/ib0pWAADAQB55SlYAAMACbW9KVgAAAA3xeUpWAAAATuZuSlYA"
+			"AIDmWXBKVgAAAAAAAAAAAABAikNwSlYAAAAAAAAAAAAAAF0pcEpWAAAAAAAAAAAAAIDv4m9KVgAA"
+			"gEAeeUpWAAAAA21vSlYAAMAM8XlKVgAAQLrDbkpWAABA5llwSlYAAAAAAAAAAAAAgIpDcEpWAAAA"
+			"AAAAAAAAAEB/K3BKVgAAAAAAAAAAAADASuNvSlYAAEDPG3lKVgAAQANtb0pWAABADfF5SlYAAICW"
+			"5m5KVgAAAPRZcEpWAAAAAAAAAAAAAMCKQ3BKVgAAAAAAAAAAAABAbytwSlYAAAAAAAAAAAAAAEjj"
+			"b0pWAABAQB55SlYAAIADbW9KVgAAgA3xeUpWAACAuMNuSlYAAED0WXBKVgAAAAAAAAAAAAAAi0Nw"
+			"SlYAAAAAAAAAAAAAgG8rcEpWAAAAAAAAAAAAAABK429KVgAAAEIeeUpWAAAABG1vSlYAAIBhi3hK"
+			"VgAAAEzmbkpWAACA9FlwSlYAAAAAAAAAAAAAQItDcEpWAAAAAAAAAAAAAAAkK3BKVgAAAAAAAAAA"
+			"AACASuNvSlYAAEBCHnlKVgAAQARtb0pWAAAAY4t4SlYAAIBO5m5KVgAAwPRZcEpWAAAAAAAAAAAA"
+			"AICLQ3BKVgAAAAAAAAAAAAAAAAAAAAAAAAAAAAAAAAAAAAAAAAAAAAAAAAAAAAAAAAAAAAAAAAAA"
+			"AAAAAAAAAAAAAAAAAAAAAAAAAAAAAAAAAAAAAAAAAAAAAAAAAAAAAAAAAAAAAAAAAAAAAAAAAAAA"
+			"AAAAAAAAAAAAAAAAAAAAAAAAAAAAAAAAAAAAAAAAAAAAAAAAAAAAAAAAAAAAAAAAAAAAAAAAAAAA"
+			"AAAAAAAAAAAAAAAAAAAAAAAAAAAAAAAAAAAAAAAAAAAAAAAAAAAAAAAAAAAAAAAAAAAAAAAAAAAA"
+			"AAAAAAAAAAAAAAAAAAAAAAAAAAAAAAAAAAAAAAAAAAAAAAAAAAAAAAAAAAAAAAAAAAAAAAAAAAAA"
+			"AAAAAAAAAAAAAAAAAAAAAAAAAAAAAAAAAAAAAAAAAAAAAAAAAAAAAAAAAAAAAAAAAAAAAAAAAAAA"
+			"AAAAAAAAAAAAAAAAAAAAAAAAAAAAAAAAAAAAAAAAAAAAAAAAAAAAAAAAAAAAAAAAAAAAAAAAAAAA"
+			"AAAAAAAAAAAAAAAAAAAAAAAAAAAAAAAAAAAAAAAAAAAAAAAAAAAAAAAAAAAAAAAAAAAAAAAAAAAA"
+			"AAAAAAAAAAAAAAAAAAAAAAAAAAAAAAAAAAAAAAAAAAAAAAAAAAAAAAAAAAAAAAAAAAAAAAAAAAAA"
+			"AAAAAAAAAAAAAAAAAAAAAAAAAAAAAAAAAAAAAAAAAAAAAAAAAAAAAAAAAAAAAAAAAAAAAAAAAAAA"
+			"AAAAAAAAAAAAAAAAAAAAAAAAAAAAAAAAAAAAAAAAAAAAAAAAAAAAAAAAAAAAAAAAAAAAAAAAAAAA"
+			"AAAAAAAAAAAAAAAAAAAAAAAAAAAAAAAAAAAAAAAAAAAAAAAAAAAAAAAAAAAAAAAAAAAAAAAAAAAA"
+			"AAAAAAAAAAAAAAAAAAAAAAAAAAAAAAAAAAAAAAAAAAAAAAAAAAAAAAAAAAAAAAAAAAAAAAAAAAAA"
+			"AAAAAAAAAAAAAAAAAAAAAAAAAAAAAAAAAAAAAAAAAAAAAAAAAAAAAAAAAAAAAAAAAAAAAAAAAAAA"
+			"AAAAAAAAAAAAAAAAAAAAAAAAAAAAAAAAAAAAAAAAAAAAAAAAAAAAAAAAAAAAAAAAAAAAAAAAAAAA"
+			"AAAAAAAAAAAAAAAAAAAAAAAAAAAAAAAAAAAAAAAAAAAAAAAAAAAAAAAAAAAAAAAAAAAAAAAAAAAA"
+			"AAAAAAAAAAAAAAAAAAAAAAAAAAAAAAAAAAAAAAAAAAAAAAAAAAAAAAAAAAAAAAAAAAAAAAAAAAAA"
+			"AAAAAAAAAAAAAAAAAAAAAAAAAAAAAAAAAAAAAAAAAAAAAAAAAAAAAAAAAAAAAAAAAAAAAAAAAAAA"
+			"AAAAAAAAAAAAAAAAAAAAAAAAAA=="
 		)
 	)
@@
 		)
 	)
-	(label "GPIO_16"
-		(at 219.71 127 0)
-		(effects
-			(font
-				(size 1.27 1.27)
-			)
-			(justify left bottom)
-		)
-	)
 	(label "5V"
 		(at 314.96 55.88 0)
@@
 		)
 	)
-	(label "GPIO_4"
-		(at 219.71 124.46 0)
-		(effects
-			(font
-				(size 1.27 1.27)
-			)
-			(justify left bottom)
-		)
-	)
 	(label "3V3"
 		(at 232.41 40.64 0)
@@
 		)
 	)
+	(label "GPIO_16"
+		(at 176.53 140.97 180)
+		(effects
+			(font
+				(size 1.27 1.27)
+			)
+			(justify right bottom)
+		)
+	)
 	(label "GPIO_4"
 		(at 270.51 254 0)
@@
 		)
 	)
+	(label "GPIO_4"
+		(at 176.53 143.51 180)
+		(effects
+			(font
+				(size 1.27 1.27)
+			)
+			(justify right bottom)
+		)
+	)
 	(label "3V3"
 		(at 165.1 138.43 0)
@@
 			)
 		)
-		(property "Footprint" "Connector_PinHeader_2.00mm:PinHeader_2x03_P2.00mm_Vertical"
+		(property "Footprint" "Connector_PinHeader_2.54mm:PinHeader_2x03_P2.54mm_Vertical"
 			(at 262.89 254 0)
 			(effects
@@
 		)
 	)
+	(embedded_fonts no)
 )
